File: Matriz_8x8.brd (EAGLE design)
At the start: 68.6 x 53.3 mm, 137 parts

Commit message: implementacion de todo el codigo recopilado
Parts:
- removed D64: (no value), AUTODESK_CIRCUITS_BREADBOARD:LED5MM
- removed U11: (no value), AUTODESK_CIRCUITS_BREADBOARD:DIL16
- added D3.8: (no value), AUTODESK_CIRCUITS_BREADBOARD:LED5MM
- added U1: (no value), AUTODESK_CIRCUITS_BREADBOARD:DIL16
- moved D1 12.7 mm to (5.00, 924.5)
- moved D2 12.7 mm to (5.00, 937.2)
- moved D3 12.7 mm to (5.00, 949.9)
- moved D4 12.7 mm to (5.00, 962.6)
- moved D5 12.7 mm to (5.00, 975.3)
- moved D6 12.7 mm to (5.00, 988.0)
- moved D7 12.7 mm to (5.00, 1000.7)
- moved D8 12.7 mm to (5.00, 1013.4)
- moved R5.1 12.7 mm to (5.00, 518.1)
- moved R5.2 12.7 mm to (5.00, 530.8)
- moved R5.3 12.7 mm to (5.00, 543.5)
- moved R5.4 12.7 mm to (5.00, 556.2)
- moved R5.5 12.7 mm to (5.00, 568.9)
- moved R5.6 12.7 mm to (5.00, 581.6)
- moved R5.7 12.7 mm to (5.00, 594.3)
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- renumbered D41 to D3.7, D42 to D3.6, D43 to D3.5, D44 to D3.4, D45 to D3.3, D46 to D3.2, D47 to D3.1, D48 to D2.8, D49 to D2.7, D50 to D2.6, D51 to D2.5, D52 to D2.4, D53 to D2.3, D54 to D2.2, D55 to D2.1, D56 to D1.8, D57 to D1.7, D58 to D1.6, D59 to D1.5, D60 to D1.4, D61 to D1.3, D62 to D1.2, D63 to D1.1
Connections:
- removed net N$100 (its old number): D3.4.A, R3.5.2
- removed net N$101 (its old number): D3.5.A, R3.6.2
- removed net N$102 (its old number): D3.6.A, R3.7.2
- removed net N$103 (its old number): D3.7.A, R3.8.2
- removed net N$73 (its old number): D1.1.K, D1.2.K, D1.3.K, D1.4.K, D1.5.K, D1.6.K, D1.7.K, D1.8.K, D1.K, D10.K, D11.K, D12.K, D13.K, D14.K, D15.K, D16.K, D17.K, D18.K, D19.K, D2.1.K, D2.2.K, D2.3.K, D2.4.K, D2.5.K, D2.6.K, D2.7.K, D2.8.K, D2.K, D20.K, D21.K, D22.K, D23.K, D24.K, D25.K, D26.K, D27.K, D28.K, D29.K, D3.1.K, D3.2.K, D3.3.K, D3.4.K, D3.5.K, D3.6.K, D3.7.K, D3.K, D30.K, D31.K, D32.K, D33.K, D34.K, D35.K, D36.K, D37.K, D38.K, D39.K, D4.K, D40.K, D5.K, D6.K, D64.K, D7.K, D8.K, D9.K, U10.13, U10.8, U11.13, U11.8, U12.13, U12.8, U13.13, U13.8, U14.13, U14.8, U16.13, U16.8, U17.13, U17.8, U5.GND.., U9.13, U9.8
- new net N$140: D1.1.K, D1.2.K, D1.3.K, D1.4.K, D1.5.K, D1.6.K, D1.7.K, D1.8.K, D1.K, D10.K, D11.K, D12.K, D13.K, D14.K, D15.K, D16.K, D17.K, D18.K, D19.K, D2.1.K, D2.2.K, D2.3.K, D2.4.K, D2.5.K, D2.6.K, D2.7.K, D2.8.K, D2.K, D20.K, D21.K, D22.K, D23.K, D24.K, D25.K, D26.K, D27.K, D28.K, D29.K, D3.1.K, D3.2.K, D3.3.K, D3.4.K, D3.5.K, D3.6.K, D3.7.K, D3.8.K, D3.K, D30.K, D31.K, D32.K, D33.K, D34.K, D35.K, D36.K, D37.K, D38.K, D39.K, D4.K, D40.K, D5.K, D6.K, D7.K, D8.K, D9.K, U1.13, U1.8, U10.13, U10.8, U12.13, U12.8, U13.13, U13.8, U14.13, U14.8, U16.13, U16.8, U17.13, U17.8, U5.GND.., U9.13, U9.8
- new net N$141: D1.5.A, R1.5.2
- new net N$142: D3.5.A, R3.5.2
- new net N$143: D3.3.A, R3.3.2
- new net N$144: R3.2.1, U1.1
- new net N$79: D1.1.A, R1.1.2
- net N$1: now also U1.5; no longer R3.2.1, U11.1, U11.5
- net N$12: now also U1.11; no longer U11.11
- net N$18: now also U1.14; no longer U11.14
- net N$25: now also U1.4; no longer U11.4
- net N$26: now also U1.6; no longer U11.6
- net N$27: now also U1.7; no longer U11.7
- net N$28: now also U1.15; no longer U11.15
- net N$29: now also U1.3; no longer U11.3
- net N$30: now also U1.9; no longer U11.9
- net N$48: now also U1.10, U1.16; no longer U11.10, U11.16
- net N$50: now also U1.2; no longer U11.2
- net N$6: now also U1.12; no longer U11.12
- net N$80: now also D1.2.A, R1.2.2; no longer D64.A, R1.1.2
- net N$81: now also D1.3.A, R1.3.2; no longer D1.1.A, R1.2.2
- net N$82: now also D1.4.A, R1.4.2; no longer D1.2.A, R1.3.2
- net N$83: now also D1.6.A, R1.6.2; no longer D1.3.A, R1.4.2
- net N$84: now also D1.7.A, R1.7.2; no longer D1.4.A, R1.5.2
- net N$85: now also D1.8.A, R1.8.2; no longer D1.5.A, R1.6.2
- net N$86: now also D2.1.A, R2.1.2; no longer D1.6.A, R1.7.2
- net N$87: now also D2.2.A, R2.2.2; no longer D1.7.A, R1.8.2
- net N$88: now also D2.3.A, R2.3.2; no longer D1.8.A, R2.1.2
- net N$89: now also D2.4.A, R2.4.2; no longer D2.1.A, R2.2.2
- net N$90: now also D2.5.A, R2.5.2; no longer D2.2.A, R2.3.2
- net N$91: now also D2.6.A, R2.6.2; no longer D2.3.A, R2.4.2
- net N$92: now also D2.7.A, R2.7.2; no longer D2.4.A, R2.5.2
- net N$93: now also D2.8.A, R2.8.2; no longer D2.5.A, R2.6.2
- net N$94: now also D3.1.A, R3.1.2; no longer D2.6.A, R2.7.2
- net N$95: now also D3.2.A, R3.2.2; no longer D2.7.A, R2.8.2
- net N$96: now also D3.4.A, R3.4.2; no longer D2.8.A, R3.1.2
- net N$97: now also D3.6.A, R3.6.2; no longer D3.1.A, R3.2.2
- net N$98: now also D3.7.A, R3.7.2; no longer D3.2.A, R3.3.2
- net N$99: now also D3.8.A, R3.8.2; no longer D3.3.A, R3.4.2
